Commit message: changed frames in turtlebot3

File: install/turtlebot3_gazebo/share/turtlebot3_gazebo/urdf/turtlebot3_waffle_pi.urdf (robot description, URDF)
Before this commit: robot turtlebot3_waffle_pi, 11 links, 10 joints
Links:
- removed link camera_rgb_optical_frame
- added link camera_color_optical_frame
Joints:
- joint camera_rgb_optical_joint: child camera_rgb_optical_frame -> camera_color_optical_frame
